File: soar-noflash.brd (EAGLE design)
At the start: 55.6 x 19.9 mm, 27 parts, among them IC3 MCP1703CB, U2 9DoF IMU, U3 915MHz, U6 BME280, X1 16 MHz

Commit message: in progress
Parts:
- removed U$6: AT25F512BWIDE_5.3MM, LowPowerLab:SO08WIDE
Connections:
- net D11_MOSI: no longer U$6.5
- net D12_MISO: no longer U$6.2
- net D13_SCK: no longer U$6.6
- net D8: no longer U$6.1
- net GND: no longer U$6.4
- net VCC: no longer U$6.3, U$6.7, U$6.8
Changed lines of the file:
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@@
 <element name="U$2" library="LowPowerLab" package="0603-LED" value="LED0603" x="72.910703125" y="43.30826875"/>
 <element name="U$3" library="LowPowerLab" package="RFM12B-ANTENNA" value="RFM12B_ANTENNA" x="25.232359375" y="42.882815625"/>
-<element name="U$6" library="LowPowerLab" package="SO08WIDE" value="AT25F512BWIDE_5.3MM" x="64.33185" y="50.622203125" rot="R180"/>
 <element name="U2" library="SparkFun-Sensors" package="QFN24-3X3" value="9DoF IMU" x="40.34409375" y="50.90668125" smashed="yes" rot="R180">
 <attribute name="NAME" x="40.34409375" y="48.87468125" size="0.6096" layer="25" font="vector" ratio="20" rot="R180" align="bottom-center"/>
@@
 <contactref element="C5" pad="2"/>
 <contactref element="U$2" pad="MINUS"/>
-<contactref element="U$6" pad="4"/>
 <contactref element="U6" pad="1"/>
 <contactref element="U6" pad="7"/>
@@
 <wire x1="67.801490625" y1="58.76708125" x2="71.4146" y2="56.69008125" width="0" layer="19" extent="1-1"/>
 <wire x1="74.382628125" y1="51.958746875" x2="71.4146" y2="56.69008125" width="0" layer="19" extent="1-1"/>
-<wire x1="62.42685" y1="53.890903125" x2="67.801490625" y2="58.76708125" width="0" layer="19" extent="1-1"/>
-<wire x1="58.923290625" y1="53.666390625" x2="62.42685" y2="53.890903125" width="0" layer="19" extent="1-1"/>
+<wire x1="60.44475" y1="57.541159375" x2="67.801490625" y2="58.76708125" width="0" layer="19" extent="1-1"/>
+<wire x1="58.923290625" y1="53.666390625" x2="60.44475" y2="57.541159375" width="0" layer="19" extent="1-1"/>
 <wire x1="59.04775" y1="50.220878125" x2="58.923290625" y2="53.666390625" width="0" layer="19" extent="1-1"/>
 <wire x1="59.238390625" y1="47.34433125" x2="59.04775" y2="50.220878125" width="0" layer="19" extent="1-1"/>
-<wire x1="60.44475" y1="57.541159375" x2="62.42685" y2="53.890903125" width="0" layer="19" extent="1-1"/>
 <wire x1="53.569865625" y1="50.02671875" x2="59.04775" y2="50.220878125" width="0" layer="19" extent="1-1"/>
 <wire x1="53.569865625" y1="51.62671875" x2="53.569865625" y2="50.02671875" width="0" layer="19" extent="1-1"/>
@@
 <contactref element="C4" pad="1"/>
 <contactref element="C3" pad="1"/>
-<contactref element="U$6" pad="7"/>
-<contactref element="U$6" pad="8"/>
-<contactref element="U$6" pad="3"/>
 <contactref element="U3" pad="2"/>
 <contactref element="C9" pad="1"/>
@@
 <wire x1="67.801490625" y1="57.06708125" x2="73.3146" y2="56.69008125" width="0" layer="19" extent="1-1"/>
 <wire x1="64.65061875" y1="57.119146875" x2="67.801490625" y2="57.06708125" width="0" layer="19" extent="1-1"/>
-<wire x1="63.69685" y1="53.890903125" x2="64.65061875" y2="57.119146875" width="0" layer="19" extent="1-1"/>
-<wire x1="64.96685" y1="47.336003125" x2="63.69685" y2="53.890903125" width="0" layer="19" extent="1-1"/>
-<wire x1="66.23685" y1="47.336003125" x2="64.96685" y2="47.336003125" width="0" layer="19" extent="1-1"/>
-<wire x1="68.743828125" y1="43.10596875" x2="66.23685" y2="47.336003125" width="0" layer="19" extent="1-1"/>
-<wire x1="57.34775" y1="50.220878125" x2="63.69685" y2="53.890903125" width="0" layer="19" extent="1-1"/>
+<wire x1="57.34775" y1="50.220878125" x2="64.65061875" y2="57.119146875" width="0" layer="19" extent="1-1"/>
 <wire x1="57.238390625" y1="47.34433125" x2="57.34775" y2="50.220878125" width="0" layer="19" extent="1-1"/>
 <wire x1="53.569865625" y1="50.82671875" x2="57.34775" y2="50.220878125" width="0" layer="19" extent="1-1"/>
@@
 <wire x1="38.707828125" y1="43.722909375" x2="41.89659375" y2="49.90668125" width="0" layer="19" extent="1-16"/>
 <wire x1="46.54079375" y1="43.82896875" x2="41.89659375" y2="49.90668125" width="0" layer="19" extent="1-1"/>
+<wire x1="68.743828125" y1="43.10596875" x2="57.238390625" y2="47.34433125" width="0" layer="19" extent="1-1"/>
 </signal>
 <signal name="D9">
@@
 <signal name="D8">
 <contactref element="ATMEGA328" pad="12"/>
-<contactref element="U$6" pad="1"/>
-<wire x1="49.677265625" y1="55.51931875" x2="66.23685" y2="53.890903125" width="0" layer="19" extent="1-1"/>
 </signal>
 <signal name="D7">
@@
 <signal name="D11_MOSI">
 <contactref element="ATMEGA328" pad="15"/>
-<contactref element="U$6" pad="5"/>
 <contactref element="U3" pad="5"/>
-<wire x1="47.277265625" y1="55.51931875" x2="62.42685" y2="47.336003125" width="0" layer="19" extent="1-1"/>
 <wire x1="32.707828125" y1="43.722909375" x2="47.277265625" y2="55.51931875" width="0" layer="19" extent="1-16"/>
 </signal>
 <signal name="D12_MISO">
 <contactref element="ATMEGA328" pad="16"/>
-<contactref element="U$6" pad="2"/>
 <contactref element="U3" pad="8"/>
-<wire x1="46.477265625" y1="55.51931875" x2="64.96685" y2="53.890903125" width="0" layer="19" extent="1-1"/>
 <wire x1="28.707828125" y1="58.722909375" x2="46.477265625" y2="55.51931875" width="0" layer="19" extent="1-16"/>
 </signal>
 <signal name="D13_SCK">
 <contactref element="ATMEGA328" pad="17"/>
-<contactref element="U$6" pad="6"/>
 <contactref element="U3" pad="6"/>
-<wire x1="44.984665625" y1="54.02671875" x2="63.69685" y2="47.336003125" width="0" layer="19" extent="1-1"/>
 <wire x1="30.707828125" y1="43.722909375" x2="44.984665625" y2="54.02671875" width="0" layer="19" extent="1-16"/>
 </signal>
